File: Polyg/hardware/Board-Back.brd (EAGLE design)
At the start: 40.1 x 109.7 mm, 45 parts, among them IC1 7805DT, U1 TL074_SMD, U3 TEENSY_3.1_BASIC, U4 CS4334

Commit message: Add files via upload
Parts:
- removed C4: 4.7µ, resistor:153CLV-0405
- added C3: 3.3n, resistor:C1206
- GAIN: value 50k -> 10k
- R10, R11, R12, R13, R15, R16: value 2k -> 220
Connections:
- new net N$2: U3.A14
- new net N$6: U3.20/A6
- net GND: now also C3.2; no longer C4.-
- net N$11: now also C3.1; no longer C4.+
Other:
- outline, holes or cut-outs redrawn
Changed lines of the file:
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@@
 <grid distance="1.27" unitdist="mm" unit="inch" style="lines" multiple="1" display="yes" altdistance="5" altunitdist="mil" altunit="inch"/>
 <layers>
-<layer number="1" name="Top" color="4" fill="1" visible="no" active="yes"/>
+<layer number="1" name="Top" color="4" fill="1" visible="yes" active="yes"/>
 <layer number="2" name="Route2" color="1" fill="3" visible="no" active="no"/>
 <layer number="3" name="Route3" color="4" fill="3" visible="no" active="no"/>
@@
 <layer number="14" name="Route14" color="1" fill="6" visible="no" active="no"/>
 <layer number="15" name="Route15" color="4" fill="6" visible="no" active="no"/>
-<layer number="16" name="Bottom" color="1" fill="1" visible="no" active="yes"/>
+<layer number="16" name="Bottom" color="1" fill="1" visible="yes" active="yes"/>
 <layer number="17" name="Pads" color="2" fill="1" visible="yes" active="yes"/>
 <layer number="18" name="Vias" color="2" fill="1" visible="yes" active="yes"/>
@@
 <wire x1="0" y1="109.652" x2="0" y2="0" width="0" layer="20"/>
 <wire x1="0" y1="0" x2="40.14" y2="0" width="0" layer="20"/>
-<wire x1="40.14" y1="0" x2="39.886" y2="109.652" width="0" layer="20"/>
-<wire x1="39.886" y1="109.652" x2="0" y2="109.652" width="0" layer="20"/>
+<wire x1="40.14" y1="0" x2="40.14" y2="109.652" width="0" layer="20"/>
+<wire x1="40.14" y1="109.652" x2="0" y2="109.652" width="0" layer="20"/>
 <text x="6.5405" y="83.8835" size="1.778" layer="21" font="vector" rot="MR0">RED</text>
 <hole x="6.35" y="8.001" drill="3"/>
@@
 <attribute name="VALUE" x="21.844" y="6.35" size="1.27" layer="28" rot="MR180"/>
 </element>
-<element name="R10" library="resistor" library_urn="urn:adsk.eagle:library:348" package="M1206" package3d_urn="urn:adsk.eagle:package:26088/1" value="2k" x="15.494" y="73.152" smashed="yes" rot="MR180">
+<element name="R10" library="resistor" library_urn="urn:adsk.eagle:library:348" package="M1206" package3d_urn="urn:adsk.eagle:package:26088/1" value="220" x="15.494" y="73.152" smashed="yes" rot="MR180">
 <attribute name="NAME" x="10.414" y="73.787" size="1.27" layer="26" rot="MR180"/>
 <attribute name="VALUE" x="14.224" y="75.692" size="1.27" layer="28" rot="MR180"/>
 </element>
-<element name="R11" library="resistor" library_urn="urn:adsk.eagle:library:348" package="M1206" package3d_urn="urn:adsk.eagle:package:26088/1" value="2k" x="15.494" y="69.85" smashed="yes" rot="MR180">
+<element name="R11" library="resistor" library_urn="urn:adsk.eagle:library:348" package="M1206" package3d_urn="urn:adsk.eagle:package:26088/1" value="220" x="15.494" y="69.85" smashed="yes" rot="MR180">
 <attribute name="NAME" x="10.7315" y="70.485" size="1.27" layer="26" rot="MR180"/>
 <attribute name="VALUE" x="14.224" y="72.39" size="1.27" layer="28" rot="MR180"/>
 </element>
-<element name="R12" library="resistor" library_urn="urn:adsk.eagle:library:348" package="M1206" package3d_urn="urn:adsk.eagle:package:26088/1" value="2k" x="15.494" y="66.548" smashed="yes" rot="MR180">
+<element name="R12" library="resistor" library_urn="urn:adsk.eagle:library:348" package="M1206" package3d_urn="urn:adsk.eagle:package:26088/1" value="220" x="15.494" y="66.548" smashed="yes" rot="MR180">
 <attribute name="NAME" x="10.414" y="67.183" size="1.27" layer="26" rot="MR180"/>
 <attribute name="VALUE" x="14.224" y="69.088" size="1.27" layer="28" rot="MR180"/>
 </element>
-<element name="R13" library="resistor" library_urn="urn:adsk.eagle:library:348" package="M1206" package3d_urn="urn:adsk.eagle:package:26088/1" value="2k" x="15.494" y="63.246" smashed="yes" rot="MR180">
+<element name="R13" library="resistor" library_urn="urn:adsk.eagle:library:348" package="M1206" package3d_urn="urn:adsk.eagle:package:26088/1" value="220" x="15.494" y="63.246" smashed="yes" rot="MR180">
 <attribute name="NAME" x="10.7315" y="63.881" size="1.27" layer="26" rot="MR180"/>
 <attribute name="VALUE" x="14.224" y="65.786" size="1.27" layer="28" rot="MR180"/>
 </element>
-<element name="R15" library="resistor" library_urn="urn:adsk.eagle:library:348" package="M1206" package3d_urn="urn:adsk.eagle:package:26088/1" value="2k" x="15.494" y="56.642" smashed="yes" rot="MR180">
+<element name="R15" library="resistor" library_urn="urn:adsk.eagle:library:348" package="M1206" package3d_urn="urn:adsk.eagle:package:26088/1" value="220" x="15.494" y="56.642" smashed="yes" rot="MR180">
 <attribute name="NAME" x="10.0965" y="57.277" size="1.27" layer="26" rot="MR180"/>
 <attribute name="VALUE" x="14.224" y="59.182" size="1.27" layer="28" rot="MR180"/>
 </element>
-<element name="R16" library="resistor" library_urn="urn:adsk.eagle:library:348" package="M1206" package3d_urn="urn:adsk.eagle:package:26088/1" value="2k" x="15.494" y="53.34" smashed="yes" rot="MR180">
+<element name="R16" library="resistor" library_urn="urn:adsk.eagle:library:348" package="M1206" package3d_urn="urn:adsk.eagle:package:26088/1" value="220" x="15.494" y="53.34" smashed="yes" rot="MR180">
 <attribute name="NAME" x="12.954" y="52.07" size="1.27" layer="26" rot="MR180"/>
 <attribute name="VALUE" x="14.224" y="55.88" size="1.27" layer="28" rot="MR180"/>
@@
 <attribute name="VALUE" x="25.019" y="51.308" size="1.27" layer="27" rot="R180"/>
 </element>
-<element name="GAIN" library="MusicThingModular" package="BOURNS_3362P_TRIMMER" value="50k" x="34.036" y="28.702" smashed="yes" rot="MR0">
+<element name="GAIN" library="MusicThingModular" package="BOURNS_3362P_TRIMMER" value="10k" x="34.036" y="28.702" smashed="yes" rot="MR0">
 <attribute name="NAME" x="37.6555" y="23.4315" size="1.27" layer="26" ratio="10" rot="MR0"/>
 <attribute name="VALUE" x="37.3126" y="23.495" size="1.27" layer="28" ratio="10" rot="MR0"/>
@@
 <attribute name="VALUE" x="16.002" y="46.736" size="1.27" layer="27" rot="R180"/>
 </element>
-<element name="C4" library="resistor" library_urn="urn:adsk.eagle:library:348" package="153CLV-0405" package3d_urn="urn:adsk.eagle:package:25891/1" value="4.7µ" x="9.906" y="47.752" smashed="yes">
-<attribute name="NAME" x="5.4435" y="47.3745" size="1.27" layer="25"/>
-<attribute name="VALUE" x="7.631" y="44.017" size="1.27" layer="27"/>
-</element>
+<element name="C3" library="resistor" library_urn="urn:adsk.eagle:library:348" package="C1206" package3d_urn="urn:adsk.eagle:package:26140/1" value="3.3n" x="10.16" y="48.26" rot="R180"/>
 </elements>
 <signals>
@@
 <contactref element="R6" pad="2"/>
 <contactref element="R2" pad="2"/>
-<contactref element="C4" pad="-"/>
+<contactref element="C3" pad="2"/>
 </signal>
 <signal name="+3.3V">
@@
 <signal name="N$11">
 <contactref element="R14" pad="2"/>
-<contactref element="C4" pad="+"/>
 <contactref element="R3" pad="1"/>
 <contactref element="U1" pad="12"/>
@@
 <wire x1="17.72" y1="42.418" x2="19.244" y2="44.196" width="0.4064" layer="1"/>
 <wire x1="19.244" y1="44.196" x2="20.514" y2="44.196" width="0.4064" layer="1"/>
-<wire x1="11.706" y1="47.752" x2="13.462" y2="46.25" width="0.4064" layer="1"/>
-<wire x1="13.462" y1="46.25" x2="13.462" y2="44.958" width="0.4064" layer="1"/>
 <wire x1="24.511" y1="53.086" x2="29.08" y2="53.086" width="0.3048" layer="1"/>
 <wire x1="22.43074375" y1="44.35536875" x2="22.908" y2="44.832625" width="0.3048" layer="1"/>
 <wire x1="22.908" y1="44.832625" x2="22.908" y2="51.483" width="0.3048" layer="1"/>
 <wire x1="22.908" y1="51.483" x2="24.511" y2="53.086" width="0.3048" layer="1"/>
+<contactref element="C3" pad="1"/>
+<wire x1="11.56" y1="48.26" x2="13.462" y2="46.358" width="0.4064" layer="1"/>
+<wire x1="13.462" y1="46.358" x2="13.462" y2="44.958" width="0.4064" layer="1"/>
+</signal>
+<signal name="N$2">
+<contactref element="U3" pad="A14"/>
+</signal>
+<signal name="N$6">
+<contactref element="U3" pad="20/A6"/>
 </signal>
 </signals>
