File: Polyg/hardware/Board-Back.brd (EAGLE design)
At the start: 40.1 x 109.7 mm, 45 parts, among them IC1 7805DT, U1 TL074_SMD, U3 TEENSY_3.1_BASIC, U4 CS4334

Commit message: Add files via upload
Parts:
- R8, R9: value 47 -> 1k
- moved IC1 2.54 mm to (14.2, 92.5)
- moved D2 1.27 mm to (7.11, 100.8)
Routing:
- net GND: track 40.2 -> 19.5 mm
- net N$9: track 4.83 -> 6.10 mm
- net +5V: track 164.9 -> 165.6 mm
- net PIN15/A1: track 37.5 -> 37.0 mm
Other:
- board text added: "+12V"
- board text added: "-12V"
- board text added: "GND"
- board text added: "Red stripe here"
- board text removed: "RED"
