File: Polyg/hardware/Frontpanel.brd (EAGLE design)
At the start: 40.1 x 127.9 mm, 0 parts

Commit message: Add files via upload
Routing:
- net DFGD: track 64.5 -> 0.00 mm
Other:
- board text added: "AUDIO"
- board text added: "GATE"
- board text added: "TRIG"
- board text added: "WAVE"
- board text removed: "AUD OUT"
- board text removed: "FM CV"
- board text removed: "GATE OUT"
- board text removed: "RATIO CV"
- board text removed: "WAVESH TRIG"
