File: Polyg/hardware/Board-Front.sch (EAGLE design)
At the start: 44 parts, among them T1 BC847

Commit message: Add files via upload
Parts:
- renumbered D1 to D10, D4 to D11, D5 to D12, R1 to R18, R10 to R19, R11 to R20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
