File: Polyg/hardware/Board-Front.brd (EAGLE design)
At the start: 40.1 x 109.4 mm, 44 parts, among them T1 BC847

Commit message: Add files via upload
Other:
- board text added: "+"
Changed lines of the file:
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@@
 <layer number="21" name="tPlace" color="7" fill="1" visible="yes" active="yes"/>
 <layer number="22" name="bPlace" color="7" fill="1" visible="yes" active="yes"/>
-<layer number="23" name="tOrigins" color="15" fill="1" visible="no" active="yes"/>
+<layer number="23" name="tOrigins" color="15" fill="1" visible="yes" active="yes"/>
 <layer number="24" name="bOrigins" color="15" fill="1" visible="yes" active="yes"/>
-<layer number="25" name="tNames" color="7" fill="1" visible="no" active="yes"/>
+<layer number="25" name="tNames" color="7" fill="1" visible="yes" active="yes"/>
 <layer number="26" name="bNames" color="7" fill="1" visible="yes" active="yes"/>
 <layer number="27" name="tValues" color="7" fill="1" visible="no" active="yes"/>
@@
 <wire x1="40.14" y1="0" x2="40.14" y2="109.398" width="0" layer="20"/>
 <wire x1="40.14" y1="109.398" x2="0" y2="109.398" width="0" layer="20"/>
+<text x="34.163" y="60.325" size="1.778" layer="25">+</text>
+<text x="29.337" y="60.579" size="1.778" layer="25">+</text>
+<text x="10.16" y="54.483" size="1.778" layer="25">+</text>
+<text x="5.334" y="54.356" size="1.778" layer="25">+</text>
+<text x="5.334" y="66.421" size="1.778" layer="25">+</text>
+<text x="10.16" y="66.421" size="1.778" layer="25">+</text>
 </plain>
 <attributes>

Commit message: Add files via upload
Parts:
- renumbered D1 to D10, D4 to D11, D5 to D12, R1 to R18, R10 to R19, R11 to R20, R12 to R29, R13 to R30, R14 to R31, R15 to R32, R16 to R33, R2 to R21, R3 to R22, R4 to R23, R5 to R24, R6 to R25, R7 to R26, R8 to R27, R9 to R28, SV2 to SV6, SV3 to SV5, SV4 to SV7

Commit message: Add files via upload
Parts:
- R26: value 1k -> 220
Changed lines of the file:
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@@
 <attribute name="VALUE" x="28.194" y="18.034" size="1.27" layer="28" rot="MR90"/>
 </element>
-<element name="R26" library="resistor" library_urn="urn:adsk.eagle:library:348" package="M1206" package3d_urn="urn:adsk.eagle:package:26088/1" value="1k" x="23.876" y="47.498" smashed="yes" rot="MR270">
+<element name="R26" library="resistor" library_urn="urn:adsk.eagle:library:348" package="M1206" package3d_urn="urn:adsk.eagle:package:26088/1" value="220" x="23.876" y="47.498" smashed="yes" rot="MR270">
 <attribute name="NAME" x="22.86" y="51.562" size="1.27" layer="26" rot="MR180"/>
 <attribute name="VALUE" x="26.416" y="48.768" size="1.27" layer="28" rot="MR270"/>
