File: Polyg/hardware/Board-Front.brd (EAGLE design)
At the start: 40.1 x 109.4 mm, 44 parts, among them T1 BC847

Commit message: Add files via upload
Parts:
- R28: value 47 -> 1k
Changed lines of the file:
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@@
 <attribute name="VALUE" x="14.478" y="46.228" size="1.27" layer="28" rot="MR180"/>
 </element>
-<element name="R28" library="resistor" library_urn="urn:adsk.eagle:library:348" package="M1206" package3d_urn="urn:adsk.eagle:package:26088/1" value="47" x="3.81" y="19.05" smashed="yes" rot="MR270">
+<element name="R28" library="resistor" library_urn="urn:adsk.eagle:library:348" package="M1206" package3d_urn="urn:adsk.eagle:package:26088/1" value="1k" x="3.81" y="19.05" smashed="yes" rot="MR270">
 <attribute name="NAME" x="2.794" y="16.129" size="1.27" layer="26" rot="MR180"/>
 <attribute name="VALUE" x="6.35" y="20.32" size="1.27" layer="28" rot="MR270"/>
