File: MFOS 4ch Stereo Mixer/hardware/stereomix-back.sch (EAGLE design)
At the start: 27 parts, among them IC1 TL082P

Commit message: Add files via upload
Parts:
- removed SV7: (no value), con-lstb:MA04-1
- added SV4: (no value), con-lstb:MA04-1
- C10, C9: value (none) -> 100µ
Connections:
- net N$35: now also SV5.1; no longer SV7.1
- net N$36: now also SV5.2; no longer SV7.2
- net N$37: now also SV5.3; no longer SV7.3
- net N$38: now also SV5.4; no longer SV7.4
- net N$39: now also SV4.1; no longer SV5.1
- net N$40: now also SV4.2; no longer SV5.2
- net N$41: now also SV4.3; no longer SV5.3
- net N$42: now also SV4.4; no longer SV5.4
Other:
- moved on the sheet: SV5
