File: MFOS 4ch Stereo Mixer/hardware/stereomix-front.brd (EAGLE design)
At the start: 30.1 x 106.7 mm, 17 parts

Commit message: Add files via upload
Parts:
- flipped SV2 to the bottom, turned to 0 degrees
- flipped SV4 to the bottom
- flipped SV6 to the bottom
Routing:
- net GND: track 35.7 -> 24.3 mm, vias 3 -> 2
- net N$34: track 17.5 -> 11.9 mm
- net N$20: track 16.7 -> 11.3 mm
- net N$22: track 12.4 -> 16.6 mm, vias 0 -> 1
- net N$27: track 68.4 -> 66.2 mm
- net N$25: track 116.0 -> 118.0 mm
- net N$18: track 12.2 -> 13.9 mm
- net N$28: track 66.9 -> 65.7 mm
- net N$30: track 57.4 -> 56.4 mm
- net N$33: track 15.7 -> 14.9 mm
- net N$23: track 74.6 -> 75.3 mm
Other:
- board size 30.1 x 106.7 mm -> 30.4 x 106.7 mm
