File: Polyg/WRONG SILKSCREEN/Board-Back.brd (EAGLE design)
At the start: 40.1 x 109.7 mm, 45 parts, among them IC2 7805DT, U2 TEENSY_3.1_BASIC, U5 TL074_SMD, U6 CS4334

Commit message: Add files via upload
Parts:
- renumbered GAIN to GAIN1, R1 to R34
Changed lines of the file:
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@@
 </element>
 <element name="C13" library="resistor" library_urn="urn:adsk.eagle:library:348" package="C1206" package3d_urn="urn:adsk.eagle:package:26140/1" value="100n" x="28.956" y="43.688" smashed="yes" rot="MR270">
-<attribute name="NAME" x="29.591" y="47.8155" size="1.27" layer="26" rot="MR270"/>
+<attribute name="NAME" x="29.591" y="48.9585" size="1.27" layer="26" rot="MR270"/>
 <attribute name="VALUE" x="31.496" y="44.958" size="1.27" layer="28" rot="MR270"/>
 </element>
@@
 </element>
 <element name="D17" library="diode" library_urn="urn:adsk.eagle:library:210" package="DO35-7" package3d_urn="urn:adsk.eagle:package:43339/1" value="1N4148" x="21.082" y="32.004" smashed="yes">
-<attribute name="NAME" x="13.716" y="33.909" size="1.27" layer="25" ratio="10"/>
+<attribute name="NAME" x="13.97" y="29.591" size="1.27" layer="25" ratio="10"/>
 <attribute name="VALUE" x="18.796" y="29.337" size="1.27" layer="27" ratio="10"/>
 </element>
 <element name="D16" library="diode" library_urn="urn:adsk.eagle:library:210" package="DO35-7" package3d_urn="urn:adsk.eagle:package:43339/1" value="1N4148" x="21.082" y="34.544" smashed="yes" rot="R180">
-<attribute name="NAME" x="15.748" y="32.639" size="1.27" layer="25" ratio="10" rot="R180"/>
+<attribute name="NAME" x="16.383" y="33.909" size="1.27" layer="25" ratio="10" rot="R180"/>
 <attribute name="VALUE" x="23.368" y="37.211" size="1.27" layer="27" ratio="10" rot="R180"/>
 </element>
@@
 <attribute name="VALUE" x="22.86" y="11.811" size="1.27" layer="27" ratio="10" rot="R180"/>
 </element>
-<element name="R1" library="resistor" library_urn="urn:adsk.eagle:library:348" package="M1206" package3d_urn="urn:adsk.eagle:package:26088/1" value="470" x="23.114" y="3.81" smashed="yes" rot="MR180">
+<element name="R34" library="resistor" library_urn="urn:adsk.eagle:library:348" package="M1206" package3d_urn="urn:adsk.eagle:package:26088/1" value="470" x="23.114" y="3.81" smashed="yes" rot="MR180">
 <attribute name="NAME" x="24.0665" y="6.35" size="1.27" layer="26" rot="MR180"/>
 <attribute name="VALUE" x="21.844" y="6.35" size="1.27" layer="28" rot="MR180"/>
@@
 </element>
 <element name="R41" library="resistor" library_urn="urn:adsk.eagle:library:348" package="M1206" package3d_urn="urn:adsk.eagle:package:26088/1" value="267k" x="7.62" y="41.656" smashed="yes" rot="R270">
-<attribute name="NAME" x="3.7465" y="42.8625" size="1.27" layer="25"/>
+<attribute name="NAME" x="2.6035" y="42.6085" size="1.27" layer="25"/>
 <attribute name="VALUE" x="5.08" y="42.926" size="1.27" layer="27" rot="R270"/>
 </element>
@@
 </element>
 <element name="R46" library="resistor" library_urn="urn:adsk.eagle:library:348" package="M1206" package3d_urn="urn:adsk.eagle:package:26088/1" value="1k" x="35.56" y="35.687" smashed="yes" rot="R90">
-<attribute name="NAME" x="39.344471875" y="36.6620625" size="1.27" layer="25" rot="R180"/>
+<attribute name="NAME" x="38.709471875" y="40.0910625" size="1.27" layer="25" rot="R180"/>
 <attribute name="VALUE" x="38.099996875" y="34.417" size="1.27" layer="27" rot="R90"/>
 </element>
@@
 <attribute name="VALUE" x="25.019" y="51.308" size="1.27" layer="27" rot="R180"/>
 </element>
-<element name="GAIN" library="MusicThingModular" package="BOURNS_3362P_TRIMMER" value="10k" x="34.036" y="28.702" smashed="yes" rot="MR0">
+<element name="GAIN1" library="MusicThingModular" package="BOURNS_3362P_TRIMMER" value="10k" x="34.036" y="28.702" smashed="yes" rot="MR0">
 <attribute name="NAME" x="37.6555" y="23.4315" size="1.27" layer="26" ratio="10" rot="MR0"/>
 <attribute name="VALUE" x="37.3126" y="23.495" size="1.27" layer="28" ratio="10" rot="MR0"/>
@@
 <contactref element="U2" pad="3.3V"/>
 <contactref element="U2" pad="3.3V1"/>
-<contactref element="R1" pad="2"/>
+<contactref element="R34" pad="2"/>
 <contactref element="SV9" pad="8"/>
 <wire x1="24.514" y1="3.81" x2="25.654" y2="4.826" width="0.4064" layer="16"/>
@@
 <signal name="MIDI_RX">
 <contactref element="OK2" pad="6"/>
-<contactref element="R1" pad="1"/>
+<contactref element="R34" pad="1"/>
 <contactref element="U2" pad="0"/>
 <wire x1="18.034" y1="7.366" x2="18.034" y2="4.318" width="0.4064" layer="16"/>
@@
 <signal name="AUDIO">
 <contactref element="SV3" pad="2"/>
-<contactref element="GAIN" pad="3"/>
-<contactref element="GAIN" pad="2"/>
+<contactref element="GAIN1" pad="3"/>
+<contactref element="GAIN1" pad="2"/>
 <contactref element="U5" pad="14"/>
 <wire x1="34.036" y1="31.242" x2="31.496" y2="28.702" width="0.4064" layer="1"/>
@@
 <signal name="N$8">
 <contactref element="R46" pad="1"/>
-<contactref element="GAIN" pad="1"/>
+<contactref element="GAIN1" pad="1"/>
 <contactref element="U5" pad="13"/>
 <wire x1="20.514" y1="42.926" x2="19.558" y2="42.926" width="0.4064" layer="1"/>

Commit message: Add files via upload
Parts:
- renumbered C17 to C1
Changed lines of the file:
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@@
 <layer number="24" name="bOrigins" color="15" fill="1" visible="yes" active="yes"/>
 <layer number="25" name="tNames" color="7" fill="1" visible="yes" active="yes"/>
-<layer number="26" name="bNames" color="7" fill="1" visible="yes" active="yes"/>
+<layer number="26" name="bNames" color="7" fill="1" visible="no" active="yes"/>
 <layer number="27" name="tValues" color="7" fill="1" visible="no" active="yes"/>
 <layer number="28" name="bValues" color="7" fill="1" visible="no" active="yes"/>
@@
 <layer number="46" name="Milling" color="3" fill="1" visible="no" active="yes"/>
 <layer number="47" name="Measures" color="7" fill="1" visible="no" active="yes"/>
-<layer number="48" name="Document" color="7" fill="1" visible="yes" active="yes"/>
+<layer number="48" name="Document" color="7" fill="1" visible="no" active="yes"/>
 <layer number="49" name="Reference" color="7" fill="1" visible="yes" active="yes"/>
 <layer number="50" name="dxf" color="7" fill="1" visible="no" active="no"/>
@@
 </element>
 <element name="U6" library="SOIC127P600X175-8N" package="SOIC127P600X175-8N" value="CS4334" x="34.544" y="14.478" smashed="yes" rot="MR180"/>
-<element name="C17" library="resistor" library_urn="urn:adsk.eagle:library:348" package="153CLV-0405" package3d_urn="urn:adsk.eagle:package:25891/1" value="3.3µ" x="10.16" y="53.848" smashed="yes" rot="R180">
+<element name="C1" library="resistor" library_urn="urn:adsk.eagle:library:348" package="153CLV-0405" package3d_urn="urn:adsk.eagle:package:25891/1" value="3.3µ" x="10.16" y="53.848" smashed="yes" rot="R180">
 <attribute name="NAME" x="7.6375" y="54.543" size="1.27" layer="25" rot="R180"/>
 <attribute name="VALUE" x="12.435" y="57.583" size="1.27" layer="27" rot="R180"/>
@@
 <wire x1="37.084" y1="12.573" x2="37.019" y2="12.573" width="0.4064" layer="16"/>
 <wire x1="35.814" y1="1.27" x2="38.608" y2="4.064" width="0.4064" layer="16"/>
-<contactref element="C17" pad="+"/>
+<contactref element="C1" pad="+"/>
 <contactref element="R41" pad="1"/>
 <wire x1="5.712" y1="43.047" x2="5.712" y2="38.103" width="0.4064" layer="1"/>
@@
 </signal>
 <signal name="N$1">
-<contactref element="C17" pad="-"/>
+<contactref element="C1" pad="-"/>
 <contactref element="R45" pad="1"/>
 <contactref element="R50" pad="1"/>
