File: Polyg/WRONG SILKSCREEN/Board-Back.sch (EAGLE design)
At the start: 45 parts, among them IC2 7805DT, U2 TEENSY_3.1_BASIC, U5 TL074_SMD, U6 CS4334

Commit message: Add files via upload
Parts:
- renumbered GAIN to GAIN1, R1 to R34
Changed lines of the file:
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@@
 <part name="OK2" library="optocoupler" library_urn="urn:adsk.eagle:library:320" deviceset="6N138" device="" package3d_urn="urn:adsk.eagle:package:21941/1"/>
 <part name="D15" library="diode" library_urn="urn:adsk.eagle:library:210" deviceset="1N4148" device="DO35-7" package3d_urn="urn:adsk.eagle:package:43339/1" value="1N4148"/>
-<part name="R1" library="resistor" library_urn="urn:adsk.eagle:library:348" deviceset="R-EU_" device="M1206" package3d_urn="urn:adsk.eagle:package:26088/1" value="470"/>
+<part name="R34" library="resistor" library_urn="urn:adsk.eagle:library:348" deviceset="R-EU_" device="M1206" package3d_urn="urn:adsk.eagle:package:26088/1" value="470"/>
 <part name="GND3" library="supply1" library_urn="urn:adsk.eagle:library:371" deviceset="GND" device=""/>
 <part name="C3" library="resistor" library_urn="urn:adsk.eagle:library:348" deviceset="C-EU" device="C1206" package3d_urn="urn:adsk.eagle:package:26140/1" value="100n"/>
@@
 <part name="R46" library="resistor" library_urn="urn:adsk.eagle:library:348" deviceset="R-EU_" device="M1206" package3d_urn="urn:adsk.eagle:package:26088/1" value="1k"/>
 <part name="GND7" library="supply1" library_urn="urn:adsk.eagle:library:371" deviceset="GND" device=""/>
-<part name="GAIN" library="MusicThingModular" deviceset="BOURNS_3362P_TRIMMER" device="P" value="10k"/>
+<part name="GAIN1" library="MusicThingModular" deviceset="BOURNS_3362P_TRIMMER" device="P" value="10k"/>
 <part name="GND10" library="supply1" library_urn="urn:adsk.eagle:library:371" deviceset="GND" device=""/>
 <part name="C5" library="resistor" library_urn="urn:adsk.eagle:library:348" deviceset="CPOL-EU" device="E5-6" package3d_urn="urn:adsk.eagle:package:25858/1" value="100µ"/>
@@
 <attribute name="VALUE" x="-183.388" y="132.8674" size="1.778" layer="96" rot="R180"/>
 </instance>
-<instance part="R1" gate="G$1" x="-137.16" y="142.24" smashed="yes" rot="R90">
+<instance part="R34" gate="G$1" x="-137.16" y="142.24" smashed="yes" rot="R90">
 <attribute name="NAME" x="-132.842" y="147.0914" size="1.778" layer="95" rot="R180"/>
 <attribute name="VALUE" x="-132.08" y="139.954" size="1.778" layer="96" rot="R180"/>
@@
 <attribute name="VALUE" x="93.98" y="55.88" size="1.778" layer="96"/>
 </instance>
-<instance part="GAIN" gate="G$1" x="106.68" y="73.66" smashed="yes" rot="R270">
+<instance part="GAIN1" gate="G$1" x="106.68" y="73.66" smashed="yes" rot="R270">
 <attribute name="NAME" x="100.584" y="70.739" size="1.524" layer="95" ratio="10"/>
 <attribute name="VALUE" x="109.474" y="71.12" size="1.524" layer="96" ratio="10"/>
@@
 </segment>
 <segment>
-<pinref part="R1" gate="G$1" pin="2"/>
+<pinref part="R34" gate="G$1" pin="2"/>
 <wire x1="-137.16" y1="147.32" x2="-137.16" y2="149.86" width="0.1524" layer="91"/>
 <label x="-137.16" y="149.86" size="1.27" layer="95" rot="R90" xref="yes"/>
@@
 <pinref part="OK2" gate="G$1" pin="VO"/>
 <wire x1="-149.86" y1="134.62" x2="-137.16" y2="134.62" width="0.1524" layer="91"/>
-<pinref part="R1" gate="G$1" pin="1"/>
+<pinref part="R34" gate="G$1" pin="1"/>
 <wire x1="-137.16" y1="134.62" x2="-137.16" y2="137.16" width="0.1524" layer="91"/>
 <wire x1="-137.16" y1="134.62" x2="-132.08" y2="134.62" width="0.1524" layer="91"/>
@@
 <wire x1="121.92" y1="83.82" x2="127" y2="83.82" width="0.1524" layer="91"/>
 <junction x="121.92" y="83.82"/>
-<pinref part="GAIN" gate="G$1" pin="3"/>
-<pinref part="GAIN" gate="G$1" pin="2"/>
+<pinref part="GAIN1" gate="G$1" pin="3"/>
+<pinref part="GAIN1" gate="G$1" pin="2"/>
 <wire x1="106.68" y1="68.58" x2="116.84" y2="68.58" width="0.1524" layer="91"/>
 <wire x1="116.84" y1="68.58" x2="116.84" y2="73.66" width="0.1524" layer="91"/>
@@
 <wire x1="101.6" y1="73.66" x2="96.52" y2="73.66" width="0.1524" layer="91"/>
 <junction x="96.52" y="73.66"/>
-<pinref part="GAIN" gate="G$1" pin="1"/>
+<pinref part="GAIN1" gate="G$1" pin="1"/>
 <pinref part="U5" gate="D" pin="-IN"/>
 </segment>

Commit message: Add files via upload
Parts:
- renumbered C17 to C1
Changed lines of the file:
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@@
 <part name="GND17" library="supply1" library_urn="urn:adsk.eagle:library:371" deviceset="GND" device=""/>
 <part name="GND16" library="supply1" library_urn="urn:adsk.eagle:library:371" deviceset="GND" device=""/>
-<part name="C17" library="resistor" library_urn="urn:adsk.eagle:library:348" deviceset="CPOL-EU" device="153CLV-0405" package3d_urn="urn:adsk.eagle:package:25891/1" value="3.3µ"/>
+<part name="C1" library="resistor" library_urn="urn:adsk.eagle:library:348" deviceset="CPOL-EU" device="153CLV-0405" package3d_urn="urn:adsk.eagle:package:25891/1" value="3.3µ"/>
 <part name="R50" library="resistor" library_urn="urn:adsk.eagle:library:348" deviceset="R-EU_" device="M1206" package3d_urn="urn:adsk.eagle:package:26088/1" value="560"/>
 <part name="GND4" library="supply1" library_urn="urn:adsk.eagle:library:371" deviceset="GND" device=""/>
@@
 <attribute name="VALUE" x="91.44" y="0" size="1.778" layer="96"/>
 </instance>
-<instance part="C17" gate="G$1" x="27.94" y="88.9" smashed="yes" rot="R90">
+<instance part="C1" gate="G$1" x="27.94" y="88.9" smashed="yes" rot="R90">
 <attribute name="NAME" x="28.067" y="92.2274" size="1.778" layer="95" rot="R180"/>
 <attribute name="VALUE" x="28.067" y="85.8774" size="1.778" layer="96" rot="R180"/>
@@
 </segment>
 <segment>
-<pinref part="C17" gate="G$1" pin="+"/>
+<pinref part="C1" gate="G$1" pin="+"/>
 <wire x1="25.4" y1="88.9" x2="20.32" y2="88.9" width="0.1524" layer="91"/>
 <pinref part="R41" gate="G$1" pin="1"/>
@@
 <net name="N$1" class="0">
 <segment>
-<pinref part="C17" gate="G$1" pin="-"/>
+<pinref part="C1" gate="G$1" pin="-"/>
 <pinref part="R45" gate="G$1" pin="1"/>
 <wire x1="33.02" y1="88.9" x2="38.1" y2="88.9" width="0.1524" layer="91"/>
