File: Polyg/WRONG SILKSCREEN/Board-Front.brd (EAGLE design)
At the start: 40.1 x 109.4 mm, 44 parts, among them T1 BC847

Commit message: Add files via upload
Parts:
- renumbered R12 to R29
Changed lines of the file:
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@@
 <attribute name="VALUE" x="27.559" y="40.513" size="1.27" layer="28" rot="MR0"/>
 </element>
-<element name="R12" library="resistor" library_urn="urn:adsk.eagle:library:348" package="M1206" package3d_urn="urn:adsk.eagle:package:26088/1" value="10k" x="31.496" y="65.532" smashed="yes" rot="R180">
+<element name="R29" library="resistor" library_urn="urn:adsk.eagle:library:348" package="M1206" package3d_urn="urn:adsk.eagle:package:26088/1" value="10k" x="31.496" y="65.532" smashed="yes" rot="R180">
 <attribute name="NAME" x="32.766" y="63.627" size="1.27" layer="25" rot="R180"/>
 <attribute name="VALUE" x="32.766" y="68.072" size="1.27" layer="27" rot="R180"/>
@@
 <contactref element="T1" pad="2"/>
 <via x="4.572" y="85.344" extent="1-16" drill="0.35"/>
-<contactref element="R12" pad="1"/>
+<contactref element="R29" pad="1"/>
 <contactref element="R30" pad="2"/>
 <contactref element="R33" pad="2"/>
@@
 <wire x1="23.114" y1="103.632" x2="22.098" y2="104.648" width="0.4064" layer="1"/>
 <wire x1="22.098" y1="104.648" x2="22.098" y2="105.918" width="0.4064" layer="1"/>
-<contactref element="R12" pad="2"/>
+<contactref element="R29" pad="2"/>
 <wire x1="30.096" y1="65.532" x2="30.096" y2="66.4519625" width="0.4064" layer="1"/>
 <wire x1="30.096" y1="66.4519625" x2="30.000146875" y2="66.547815625" width="0.4064" layer="1"/>

Commit message: Add files via upload
Parts:
- renumbered R10 to R19
Changed lines of the file:
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@@
 <attribute name="VALUE" x="29.21" y="17.78" size="1.27" layer="27" rot="R90"/>
 </element>
-<element name="R10" library="resistor" library_urn="urn:adsk.eagle:library:348" package="M1206" package3d_urn="urn:adsk.eagle:package:26088/1" value="220" x="14.224" y="4.064" smashed="yes" rot="R90">
+<element name="R19" library="resistor" library_urn="urn:adsk.eagle:library:348" package="M1206" package3d_urn="urn:adsk.eagle:package:26088/1" value="220" x="14.224" y="4.064" smashed="yes" rot="R90">
 <attribute name="NAME" x="15.24" y="8.382" size="1.27" layer="25" rot="R180"/>
 <attribute name="VALUE" x="16.764" y="2.794" size="1.27" layer="27" rot="R90"/>
@@
 <signal name="AUDIO_F">
 <contactref element="SV5" pad="2"/>
-<contactref element="R10" pad="1"/>
+<contactref element="R19" pad="1"/>
 <wire x1="27.178" y1="105.918" x2="27.178" y2="102.362" width="0.4064" layer="16"/>
 <wire x1="27.178" y1="102.362" x2="26.67" y2="101.854" width="0.4064" layer="16"/>
@@
 </signal>
 <signal name="N$5">
-<contactref element="R10" pad="2"/>
+<contactref element="R19" pad="2"/>
 <contactref element="AUDIO-OUT" pad="P$1_TIP"/>
 <wire x1="20.276" y1="2.918" x2="20.32" y2="2.874" width="0.4064" layer="1"/>

Commit message: Add files via upload
Parts:
- removed D4: 1N4148, diode:DO35-7
- added D12: 1N4148, diode:DO35-7
- moved D11 5.08 mm to (3.30, 36.1), turned to 270 degrees
Connections:
- net +3.3V_F: now also D11.C; no longer D4.C
- net GND: now also D12.A; no longer D11.A
- net WAVE_TRIG_F: now also D11.A, D12.C; no longer D11.C, D4.A
Changed lines of the file:
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@@
 <layer number="24" name="bOrigins" color="15" fill="1" visible="yes" active="yes"/>
 <layer number="25" name="tNames" color="7" fill="1" visible="yes" active="yes"/>
-<layer number="26" name="bNames" color="7" fill="1" visible="yes" active="yes"/>
+<layer number="26" name="bNames" color="7" fill="1" visible="no" active="yes"/>
 <layer number="27" name="tValues" color="7" fill="1" visible="no" active="yes"/>
 <layer number="28" name="bValues" color="7" fill="1" visible="no" active="yes"/>
@@
 <attribute name="VALUE" x="16.891" y="35.052" size="1.27" layer="27" ratio="10" rot="R90"/>
 </element>
-<element name="D4" library="diode" library_urn="urn:adsk.eagle:library:210" package="DO35-7" package3d_urn="urn:adsk.eagle:package:43339/1" value="1N4148" x="3.302" y="36.068" smashed="yes" rot="R270">
+<element name="D11" library="diode" library_urn="urn:adsk.eagle:library:210" package="DO35-7" package3d_urn="urn:adsk.eagle:package:43339/1" value="1N4148" x="3.302" y="36.068" smashed="yes" rot="R270">
 <attribute name="NAME" x="4.826" y="38.862" size="1.27" layer="25" ratio="10"/>
 <attribute name="VALUE" x="0.635" y="38.354" size="1.27" layer="27" ratio="10" rot="R270"/>
 </element>
-<element name="D11" library="diode" library_urn="urn:adsk.eagle:library:210" package="DO35-7" package3d_urn="urn:adsk.eagle:package:43339/1" value="1N4148" x="8.382" y="36.068" smashed="yes" rot="R90">
+<element name="D12" library="diode" library_urn="urn:adsk.eagle:library:210" package="DO35-7" package3d_urn="urn:adsk.eagle:package:43339/1" value="1N4148" x="8.382" y="36.068" smashed="yes" rot="R90">
 <attribute name="NAME" x="11.938" y="33.782" size="1.27" layer="25" ratio="10" rot="R180"/>
 <attribute name="VALUE" x="11.049" y="33.782" size="1.27" layer="27" ratio="10" rot="R90"/>
@@
 </element>
 <element name="R24" library="resistor" library_urn="urn:adsk.eagle:library:348" package="M1206" package3d_urn="urn:adsk.eagle:package:26088/1" value="33k" x="29.337" y="31.115" smashed="yes" rot="MR0">
-<attribute name="NAME" x="34.163" y="30.48" size="1.27" layer="26" rot="MR0"/>
+<attribute name="NAME" x="35.433" y="30.48" size="1.27" layer="26" rot="MR0"/>
 <attribute name="VALUE" x="30.607" y="28.575" size="1.27" layer="28" rot="MR0"/>
 </element>
@@
 <contactref element="MIDI-OUT" pad="P$3_SLEEVE"/>
 <contactref element="WAVE-TRIGGER" pad="P$3_SLEEVE"/>
-<contactref element="D11" pad="A"/>
+<contactref element="D12" pad="A"/>
 <contactref element="R23" pad="2"/>
 <contactref element="FM" pad="1"/>
@@
 </signal>
 <signal name="WAVE_TRIG_F">
-<contactref element="D4" pad="A"/>
-<contactref element="D11" pad="C"/>
+<contactref element="D11" pad="A"/>
+<contactref element="D12" pad="C"/>
 <contactref element="R28" pad="1"/>
 <contactref element="SV6" pad="2"/>
@@
 <signal name="+3.3V_F">
 <contactref element="R21" pad="1"/>
-<contactref element="D4" pad="C"/>
+<contactref element="D11" pad="C"/>
 <contactref element="WAVESH" pad="P$3"/>
 <contactref element="WAVESH" pad="P$4"/>

Commit message: Add files via upload
Parts:
- R26: value 1k -> 220
Changed lines of the file:
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@@
 <attribute name="VALUE" x="28.194" y="18.034" size="1.27" layer="28" rot="MR90"/>
 </element>
-<element name="R26" library="resistor" library_urn="urn:adsk.eagle:library:348" package="M1206" package3d_urn="urn:adsk.eagle:package:26088/1" value="1k" x="23.876" y="47.498" smashed="yes" rot="MR270">
+<element name="R26" library="resistor" library_urn="urn:adsk.eagle:library:348" package="M1206" package3d_urn="urn:adsk.eagle:package:26088/1" value="220" x="23.876" y="47.498" smashed="yes" rot="MR270">
 <attribute name="NAME" x="22.86" y="51.562" size="1.27" layer="26" rot="MR180"/>
 <attribute name="VALUE" x="26.416" y="48.768" size="1.27" layer="28" rot="MR270"/>
