File: Polyg/WRONG SILKSCREEN/Board-Front.sch (EAGLE design)
At the start: 44 parts, among them T1 BC847

Commit message: Add files via upload
Parts:
- renumbered R12 to R29
Changed lines of the file:
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@@
 <part name="GND23" library="supply1" library_urn="urn:adsk.eagle:library:371" deviceset="GND" device=""/>
 <part name="T1" library="transistor" library_urn="urn:adsk.eagle:library:402" deviceset="BC847" device="" package3d_urn="urn:adsk.eagle:package:29904/2"/>
-<part name="R12" library="resistor" library_urn="urn:adsk.eagle:library:348" deviceset="R-EU_" device="M1206" package3d_urn="urn:adsk.eagle:package:26088/1" value="10k"/>
+<part name="R29" library="resistor" library_urn="urn:adsk.eagle:library:348" deviceset="R-EU_" device="M1206" package3d_urn="urn:adsk.eagle:package:26088/1" value="10k"/>
 <part name="GND21" library="supply1" library_urn="urn:adsk.eagle:library:371" deviceset="GND" device=""/>
 <part name="R30" library="resistor" library_urn="urn:adsk.eagle:library:348" deviceset="R-EU_" device="M1206" package3d_urn="urn:adsk.eagle:package:26088/1" value="*"/>
@@
 </instance>
 <instance part="T1" gate="G$1" x="-50.8" y="43.18"/>
-<instance part="R12" gate="G$1" x="-111.76" y="93.98" rot="R90"/>
+<instance part="R29" gate="G$1" x="-111.76" y="93.98" rot="R90"/>
 <instance part="GND21" gate="1" x="-111.76" y="86.36"/>
 <instance part="R30" gate="G$1" x="-205.74" y="53.34" rot="R270"/>
@@
 </segment>
 <segment>
-<pinref part="R12" gate="G$1" pin="1"/>
+<pinref part="R29" gate="G$1" pin="1"/>
 <pinref part="GND21" gate="1" pin="GND"/>
 </segment>
@@
 <wire x1="-114.3" y1="99.06" x2="-111.76" y2="99.06" width="0.1524" layer="91"/>
 <label x="-106.68" y="99.06" size="1.27" layer="95" xref="yes"/>
-<pinref part="R12" gate="G$1" pin="2"/>
+<pinref part="R29" gate="G$1" pin="2"/>
 <wire x1="-111.76" y1="99.06" x2="-106.68" y2="99.06" width="0.1524" layer="91"/>
 <junction x="-111.76" y="99.06"/>

Commit message: Add files via upload
Parts:
- renumbered R10 to R19
Changed lines of the file:
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@@
 <part name="GND22" library="supply1" library_urn="urn:adsk.eagle:library:371" deviceset="GND" device=""/>
 <part name="D10" library="diode" library_urn="urn:adsk.eagle:library:210" deviceset="1N4148" device="DO35-7" package3d_urn="urn:adsk.eagle:package:43339/1" value="1N4148"/>
-<part name="R10" library="resistor" library_urn="urn:adsk.eagle:library:348" deviceset="R-EU_" device="M1206" package3d_urn="urn:adsk.eagle:package:26088/1" value="220"/>
+<part name="R19" library="resistor" library_urn="urn:adsk.eagle:library:348" deviceset="R-EU_" device="M1206" package3d_urn="urn:adsk.eagle:package:26088/1" value="220"/>
 <part name="S1" library="switch-omron" library_urn="urn:adsk.eagle:library:377" deviceset="10-XX" device="" package3d_urn="urn:adsk.eagle:package:27496/1"/>
 <part name="SV7" library="con-lsta" library_urn="urn:adsk.eagle:library:161" deviceset="FE08-1" device="" package3d_urn="urn:adsk.eagle:package:8194/1"/>
@@
 <instance part="GND22" gate="1" x="-114.3" y="12.7"/>
 <instance part="D10" gate="G$1" x="-50.8" y="86.36"/>
-<instance part="R10" gate="G$1" x="-48.26" y="104.14"/>
+<instance part="R19" gate="G$1" x="-48.26" y="104.14"/>
 <instance part="S1" gate="1" x="-152.4" y="160.02" smashed="yes" rot="R270">
 <attribute name="NAME" x="-154.94" y="166.37" size="1.778" layer="95"/>
@@
 </segment>
 <segment>
-<pinref part="R10" gate="G$1" pin="1"/>
+<pinref part="R19" gate="G$1" pin="1"/>
 <wire x1="-53.34" y1="104.14" x2="-66.04" y2="104.14" width="0.1524" layer="91"/>
 <label x="-66.04" y="104.14" size="1.27" layer="95" rot="R180" xref="yes"/>
@@
 <net name="N$5" class="0">
 <segment>
-<pinref part="R10" gate="G$1" pin="2"/>
+<pinref part="R19" gate="G$1" pin="2"/>
 <pinref part="AUDIO-OUT" gate="G$1" pin="TIP"/>
 <wire x1="-43.18" y1="104.14" x2="-33.02" y2="104.14" width="0.1524" layer="91"/>

Commit message: Add files via upload
Parts:
- removed D4: 1N4148, diode:1N4148DO35-7
- added D12: 1N4148, diode:1N4148DO35-7
Connections:
- net +3.3V_F: now also D11.C; no longer D4.C
- net GND: now also D12.A; no longer D11.A
- net WAVE_TRIG_F: now also D11.A, D12.C; no longer D11.C, D4.A
Other:
- moved on the sheet: D11
Changed lines of the file:
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@@
 <part name="R21" library="resistor" library_urn="urn:adsk.eagle:library:348" deviceset="R-EU_" device="M1206" package3d_urn="urn:adsk.eagle:package:26088/1" value="47"/>
 <part name="R22" library="resistor" library_urn="urn:adsk.eagle:library:348" deviceset="R-EU_" device="M1206" package3d_urn="urn:adsk.eagle:package:26088/1" value="47"/>
-<part name="D4" library="diode" library_urn="urn:adsk.eagle:library:210" deviceset="1N4148" device="DO35-7" package3d_urn="urn:adsk.eagle:package:43339/1" value="1N4148"/>
 <part name="D11" library="diode" library_urn="urn:adsk.eagle:library:210" deviceset="1N4148" device="DO35-7" package3d_urn="urn:adsk.eagle:package:43339/1" value="1N4148"/>
+<part name="D12" library="diode" library_urn="urn:adsk.eagle:library:210" deviceset="1N4148" device="DO35-7" package3d_urn="urn:adsk.eagle:package:43339/1" value="1N4148"/>
 <part name="GND6" library="supply1" library_urn="urn:adsk.eagle:library:371" deviceset="GND" device=""/>
 <part name="GND7" library="supply1" library_urn="urn:adsk.eagle:library:371" deviceset="GND" device=""/>
@@
 <instance part="R21" gate="G$1" x="-195.58" y="142.24" rot="R180"/>
 <instance part="R22" gate="G$1" x="-195.58" y="134.62" rot="R180"/>
-<instance part="D4" gate="G$1" x="-111.76" y="149.86" smashed="yes" rot="R90">
+<instance part="D11" gate="G$1" x="-111.76" y="149.86" smashed="yes" rot="R90">
 <attribute name="NAME" x="-106.68" y="153.1874" size="1.778" layer="95" rot="R180"/>
 <attribute name="VALUE" x="-102.87" y="149.6314" size="1.778" layer="96" rot="R180"/>
 </instance>
-<instance part="D11" gate="G$1" x="-111.76" y="137.16" smashed="yes" rot="R90">
+<instance part="D12" gate="G$1" x="-111.76" y="137.16" smashed="yes" rot="R90">
 <attribute name="NAME" x="-107.95" y="140.4874" size="1.778" layer="95" rot="R180"/>
 <attribute name="VALUE" x="-102.87" y="134.3914" size="1.778" layer="96" rot="R180"/>
@@
 </segment>
 <segment>
-<pinref part="D11" gate="G$1" pin="A"/>
+<pinref part="D12" gate="G$1" pin="A"/>
 <pinref part="GND7" gate="1" pin="GND"/>
 <wire x1="-111.76" y1="132.08" x2="-111.76" y2="134.62" width="0.1524" layer="91"/>
@@
 <net name="WAVE_TRIG_F" class="0">
 <segment>
-<pinref part="D4" gate="G$1" pin="A"/>
+<pinref part="D11" gate="G$1" pin="A"/>
 <wire x1="-111.76" y1="142.24" x2="-111.76" y2="147.32" width="0.1524" layer="91"/>
-<pinref part="D11" gate="G$1" pin="C"/>
+<pinref part="D12" gate="G$1" pin="C"/>
 <wire x1="-111.76" y1="139.7" x2="-111.76" y2="142.24" width="0.1524" layer="91"/>
 <junction x="-111.76" y="142.24"/>
@@
 </segment>
 <segment>
-<pinref part="D4" gate="G$1" pin="C"/>
+<pinref part="D11" gate="G$1" pin="C"/>
 <wire x1="-111.76" y1="152.4" x2="-111.76" y2="157.48" width="0.1524" layer="91"/>
 <label x="-111.76" y="157.48" size="1.27" layer="95" rot="R90" xref="yes"/>

Commit message: Add files via upload
Parts:
- R26: value 1k -> 220
Changed lines of the file:
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@@
 <part name="GND11" library="supply1" library_urn="urn:adsk.eagle:library:371" deviceset="GND" device=""/>
 <part name="GATE-OUT" library="MusicThingModular" deviceset="THONKICONN" device="NEW"/>
-<part name="R26" library="resistor" library_urn="urn:adsk.eagle:library:348" deviceset="R-EU_" device="M1206" package3d_urn="urn:adsk.eagle:package:26088/1" value="1k"/>
+<part name="R26" library="resistor" library_urn="urn:adsk.eagle:library:348" deviceset="R-EU_" device="M1206" package3d_urn="urn:adsk.eagle:package:26088/1" value="220"/>
 <part name="R27" library="resistor" library_urn="urn:adsk.eagle:library:348" deviceset="R-EU_" device="M1206" package3d_urn="urn:adsk.eagle:package:26088/1" value="47"/>
 <part name="GND12" library="supply1" library_urn="urn:adsk.eagle:library:371" deviceset="GND" device=""/>
